File: Hardware/SSPS Front Panel/SSPS Front Panel.brd (EAGLE design)
At the start: 400 x 160 mm, 37 parts, among them U1 P8X32A-Q44

Commit message: figuring out LEDS
Parts:
- removed DISP17, DISP18, DISP19, DISP20, DISP21, DISP22, DISP23, DISP24, DISP25, DISP26, DISP27, DISP28, DISP29, DISP30, DISP31, DISP32: (no value), PP_LED:PSA08-11GWA
- removed DISP33, DISP34, DISP35: (no value), PP_LED:20SEG_LEDBARGRAPH
- added D1, D10, D11, D12, D13, D14, D15, D16, D2, D3, D4, D5, D6, D7, D8, D9: (no value), PP_LED:WP1043
- moved DISP10 30.0 mm to (110.0, 65.0)
- moved DISP11 30.0 mm to (90.0, 65.0)
- moved DISP12 30.0 mm to (70.0, 65.0)
- moved DISP9 30.0 mm to (130.0, 65.0)
Changed lines of the file:
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@@
 <?xml version="1.0" encoding="utf-8"?>
 <!DOCTYPE eagle SYSTEM "eagle.dtd">
-<eagle version="6.5.0">
+<eagle version="6.6.0">
 <drawing>
 <settings>
@@
 <setting verticaltext="up"/>
 </settings>
-<grid distance="10" unitdist="mm" unit="mm" style="lines" multiple="1" display="yes" altdistance="5" altunitdist="mm" altunit="mm"/>
+<grid distance="10" unitdist="mm" unit="mm" style="lines" multiple="1" display="yes" altdistance="0.25" altunitdist="mm" altunit="mm"/>
 <layers>
 <layer number="1" name="Top" color="4" fill="1" visible="yes" active="yes"/>
@@
 <element name="DISP7" library="PP_LED" package="PSA08-11GWA" value="" x="290" y="125"/>
 <element name="DISP8" library="PP_LED" package="PSA08-11GWA" value="" x="270" y="125"/>
-<element name="DISP9" library="PP_LED" package="PSA08-11GWA" value="" x="130" y="95"/>
-<element name="DISP10" library="PP_LED" package="PSA08-11GWA" value="" x="110" y="95"/>
-<element name="DISP11" library="PP_LED" package="PSA08-11GWA" value="" x="90" y="95"/>
-<element name="DISP12" library="PP_LED" package="PSA08-11GWA" value="" x="70" y="95"/>
+<element name="DISP9" library="PP_LED" package="PSA08-11GWA" value="" x="130" y="65"/>
+<element name="DISP10" library="PP_LED" package="PSA08-11GWA" value="" x="110" y="65"/>
+<element name="DISP11" library="PP_LED" package="PSA08-11GWA" value="" x="90" y="65"/>
+<element name="DISP12" library="PP_LED" package="PSA08-11GWA" value="" x="70" y="65"/>
 <element name="DISP13" library="PP_LED" package="PSA08-11GWA" value="" x="130" y="125"/>
 <element name="DISP14" library="PP_LED" package="PSA08-11GWA" value="" x="110" y="125"/>
 <element name="DISP15" library="PP_LED" package="PSA08-11GWA" value="" x="90" y="125"/>
 <element name="DISP16" library="PP_LED" package="PSA08-11GWA" value="" x="70" y="125"/>
-<element name="DISP17" library="PP_LED" package="PSA08-11GWA" value="" x="130" y="65"/>
-<element name="DISP18" library="PP_LED" package="PSA08-11GWA" value="" x="110" y="65"/>
-<element name="DISP19" library="PP_LED" package="PSA08-11GWA" value="" x="90" y="65"/>
-<element name="DISP20" library="PP_LED" package="PSA08-11GWA" value="" x="70" y="65"/>
-<element name="DISP21" library="PP_LED" package="PSA08-11GWA" value="" x="130" y="35"/>
-<element name="DISP22" library="PP_LED" package="PSA08-11GWA" value="" x="110" y="35"/>
-<element name="DISP23" library="PP_LED" package="PSA08-11GWA" value="" x="90" y="35"/>
-<element name="DISP24" library="PP_LED" package="PSA08-11GWA" value="" x="70" y="35"/>
-<element name="DISP25" library="PP_LED" package="PSA08-11GWA" value="" x="330" y="65"/>
-<element name="DISP26" library="PP_LED" package="PSA08-11GWA" value="" x="310" y="65"/>
-<element name="DISP27" library="PP_LED" package="PSA08-11GWA" value="" x="290" y="65"/>
-<element name="DISP28" library="PP_LED" package="PSA08-11GWA" value="" x="270" y="65"/>
-<element name="DISP29" library="PP_LED" package="PSA08-11GWA" value="" x="330" y="35"/>
-<element name="DISP30" library="PP_LED" package="PSA08-11GWA" value="" x="310" y="35"/>
-<element name="DISP31" library="PP_LED" package="PSA08-11GWA" value="" x="290" y="35"/>
-<element name="DISP32" library="PP_LED" package="PSA08-11GWA" value="" x="270" y="35"/>
-<element name="DISP33" library="PP_LED" package="20SEG_LEDBARGRAPH" value="" x="40" y="50"/>
-<element name="DISP34" library="PP_LED" package="20SEG_LEDBARGRAPH" value="" x="40" y="110"/>
-<element name="DISP35" library="PP_LED" package="20SEG_LEDBARGRAPH" value="" x="240" y="50"/>
 <element name="DISP36" library="PP_LED" package="20SEG_LEDBARGRAPH" value="" x="240" y="110"/>
+<element name="D1" library="PP_LED" package="WP1043" value="" x="48.31149375" y="49.91018125" rot="R80"/>
+<element name="D2" library="PP_LED" package="WP1043" value="" x="48.929703125" y="53.416109375" rot="R80"/>
+<element name="D3" library="PP_LED" package="WP1043" value="" x="49.547878125" y="56.922015625" rot="R80"/>
+<element name="D4" library="PP_LED" package="WP1043" value="" x="50.784265625" y="63.933853125" rot="R80"/>
+<element name="D5" library="PP_LED" package="WP1043" value="" x="55.77698125" y="79.40048125" rot="R50"/>
+<element name="D6" library="PP_LED" package="WP1043" value="" x="51.4024375" y="67.43978125" rot="R80"/>
+<element name="D7" library="PP_LED" package="WP1043" value="" x="52.020615625" y="70.945684375" rot="R80"/>
+<element name="D8" library="PP_LED" package="WP1043" value="" x="53.3254125" y="75.4177875" rot="R65"/>
+<element name="D9" library="PP_LED" package="WP1043" value="" x="68.04641875" y="85.89925" rot="R5"/>
+<element name="D10" library="PP_LED" package="WP1043" value="" x="63.4875625" y="84.85623125" rot="R20"/>
+<element name="D11" library="PP_LED" package="WP1043" value="" x="50.16606875" y="60.427934375" rot="R80"/>
+<element name="D12" library="PP_LED" package="WP1043" value="" x="72.307675" y="86.234640625"/>
+<element name="D13" library="PP_LED" package="WP1043" value="" x="75.867678125" y="86.234640625"/>
+<element name="D14" library="PP_LED" package="WP1043" value="" x="82.987678125" y="86.23463125"/>
+<element name="D15" library="PP_LED" package="WP1043" value="" x="79.427684375" y="86.23464375"/>
+<element name="D16" library="PP_LED" package="WP1043" value="" x="59.303684375" y="82.67775625" rot="R35"/>
 </elements>
 <signals>

Commit message: Working on Front panel.
Parts:
- removed DISP36: (no value), PP_LED:20SEG_LEDBARGRAPH
- added D100, D101, D102, D103, D104, D105, D106, D107, D108, D17, D18, D19, D20, D21, D22, D23, D24, D25, D26, D27, D28, D29, D30, D31, D32, D33, D34, D35, D36, D37, D38, D39, D40, D41, D42, D43, D44, D45, D46, D47, D48, D49, D50, D51, D52, D53, D54, D55, D56, D57, D58, D59, D60, D61, D62, D63, D64, D65, D66, D67, D68, D69, D70, D71, D72, D73, D74, D75, D76, D77, D78, D79, D80, D81, D82, D83, D84, D85, D86, D87, D88, D89, D90, D91, D92, D93, D94, D95, D96, D97, D98, D99: (no value), PP_LED:WP1043
- added DISP17, DISP18, DISP19, DISP20: PSA08-11GWA, PP_LED:PSA08-11GWA
- added SW1, SW10, SW11, SW12, SW13, SW14, SW15, SW16, SW2, SW3, SW4, SW5, SW6, SW7, SW8, SW9: B3W-9000-RG2C, PP_Electromechanical:B3W-9000
- DISP1, DISP10, DISP11, DISP12, DISP13, DISP14, DISP15, DISP16, DISP2, DISP3, DISP4, DISP5, DISP6, DISP7, DISP8, DISP9: value (none) -> PSA08-11GWA
- moved D1 96.3 mm to (42.5, 146.0), turned to 180 degrees
- moved D2 92.6 mm to (46.2, 146.0), turned to 180 degrees
- moved D11 90.3 mm to (79.0, 146.0), turned to 180 degrees
- moved D3 89.1 mm to (49.9, 146.0), turned to 180 degrees
- moved D4 82.1 mm to (53.5, 146.0), turned to 180 degrees
- moved D6 79.1 mm to (60.8, 146.0), turned to 180 degrees
- moved D7 76.1 mm to (64.5, 146.0), turned to 180 degrees
- moved D16 73.8 mm to (97.3, 146.0), turned to 180 degrees
- moved D8 72.1 mm to (68.1, 146.0), turned to 180 degrees
- moved D5 66.6 mm to (57.1, 146.0), turned to 180 degrees
- moved D10 62.3 mm to (75.4, 146.0), turned to 180 degrees
- moved D15 61.4 mm to (93.7, 146.0), turned to 180 degrees
- moved D13 60.7 mm to (86.3, 146.0), turned to 180 degrees
- moved D12 60.7 mm to (82.7, 146.0), turned to 180 degrees
- moved D9 60.2 mm to (71.8, 146.0), turned to 180 degrees
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
Commit message: Layout for front panel update.
Parts:
- added EN1, EN2: PEL12T-4226F-S1024, PP_Electromechanical:PEL12T
- added H1, H10, H2, H3, H4, H5, H6, H7, H8, H9: MOUNT_HOLE150MIL, PP_Connectors:MOUNT_HOLE_150MIL
- added LCD1: (no value), PP_Displays:CHAR_DISPLAY_1602_COUNTERSINK
- added SW17, SW18, SW19, SW20, SW21, SW22, SW23, SW24: B3W-9000-RG2C, PP_Electromechanical:B3W-9000
- added SW25, SW26: 5501M112, PP_Electromechanical:5501
- moved SW13 39.8 mm to (315.0, 70.0)
- moved SW14 38.6 mm to (328.0, 70.0)
- moved SW9 38.3 mm to (315.0, 83.0)
- moved SW15 37.4 mm to (341.0, 70.0)
- moved SW10 37.0 mm to (328.0, 83.0)
- moved SW5 36.8 mm to (315.0, 96.0)
- moved SW16 36.4 mm to (354.0, 70.0)
- moved SW11 35.8 mm to (341.0, 83.0)
- moved SW6 35.5 mm to (328.0, 96.0)
- moved SW1 35.4 mm to (315.0, 109.0)
- moved SW12 34.7 mm to (354.0, 83.0)
- moved SW7 34.2 mm to (341.0, 96.0)
- moved SW2 34.0 mm to (328.0, 109.0)
- moved SW8 33.0 mm to (354.0, 96.0)
- moved SW3 32.6 mm to (341.0, 109.0)
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Other:
- outline, holes or cut-outs redrawn
- board text added: "BINDING POSTS P/N: 6883"
- board text added: "CONNECT GROUNDS"
- board text added: "KNOB P/N: 450-KLN910"
- board text added: "PARALLIZE OUTPUTS"
- board text added: "POWER DISCONNECT P/N: 3069707"
- board text added: "SERIALIZE OUTPUTS"

Commit message: Front panel test layout almost complete.
Parts:
- removed LCD1: (no value), PP_Displays:CHAR_DISPLAY_1602_COUNTERSINK
- removed SW24: B3W-9000-RG2C, PP_Electromechanical:B3W-9000
- added DISP21: CU16025-UWJ6, PP_Displays:CU16025-UW6J
- added J1: 61400413321, PP_Connectors:61400413321
- added U2: STP16CP05XTTR, PP_DigitalIC:STP16CP05XTTR_TTSOP-24
Connections:
- new net SLD: J1.S1, J1.S2
Changed lines of the file:
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@@
 <element name="SW22" library="PP_Electromechanical" package="B3W-9000" value="B3W-9000-RG2C" x="285" y="30"/>
 <element name="SW23" library="PP_Electromechanical" package="B3W-9000" value="B3W-9000-RG2C" x="285" y="15"/>
-<element name="SW24" library="PP_Electromechanical" package="B3W-9000" value="B3W-9000-RG2C" x="-15" y="40"/>
 <element name="SW25" library="PP_Electromechanical" package="5501" value="5501M112" x="15" y="125" rot="R90"/>
 <element name="SW26" library="PP_Electromechanical" package="5501" value="5501M112" x="160" y="125" rot="R90"/>
 <element name="EN1" library="PP_Electromechanical" package="PEL12T" value="PEL12T-4226F-S1024" x="380" y="105"/>
 <element name="EN2" library="PP_Electromechanical" package="PEL12T" value="PEL12T-4226F-S1024" x="380" y="75"/>
-<element name="LCD1" library="PP_Displays" package="CHAR_DISPLAY_1602_COUNTERSINK" value="" x="305" y="155"/>
 <element name="H1" library="PP_Connectors" package="MOUNT_HOLE_150MIL" value="MOUNT_HOLE150MIL" x="5" y="5"/>
 <element name="H2" library="PP_Connectors" package="MOUNT_HOLE_150MIL" value="MOUNT_HOLE150MIL" x="5" y="155"/>
@@
 <element name="H9" library="PP_Connectors" package="MOUNT_HOLE_150MIL" value="MOUNT_HOLE150MIL" x="285" y="115"/>
 <element name="H10" library="PP_Connectors" package="MOUNT_HOLE_150MIL" value="MOUNT_HOLE150MIL" x="140" y="115"/>
+<element name="U2" library="PP_DigitalIC" package="STP16CP05XTTR_TTSOP-24" value="STP16CP05XTTR" x="40" y="130" rot="MR0"/>
+<element name="DISP21" library="PP_Displays" package="CU16025-UW6J" value="CU16025-UWJ6" x="307" y="122"/>
+<element name="J1" library="PP_Connectors" package="61400413321" value="61400413321" x="20" y="30"/>
 </elements>
 <signals>
@@
 <wire x1="-13.79" y1="129.76" x2="-20.29" y2="125.66" width="0" layer="19" extent="1-1"/>
 </signal>
+<signal name="SLD">
+<contactref element="J1" pad="S1"/>
+<contactref element="J1" pad="S2"/>
+<wire x1="26.02" y1="30" x2="13.98" y2="30" width="0" layer="19" extent="1-1"/>
+</signal>
 </signals>

Commit message: Working on front panel.
Parts:
- removed SW22, SW23: B3W-9000-RG2C, PP_Electromechanical:B3W-9000
- removed SW25, SW26: 5501M112, PP_Electromechanical:5501
- DISP1, DISP10, DISP11, DISP12, DISP13, DISP14, DISP15, DISP16, DISP17, DISP18, DISP19, DISP2, DISP20, DISP3, DISP4, DISP5, DISP6, DISP7, DISP8, DISP9: device PP_LED:PSA08-11GWA -> PP_LED:PSA08-11SRWA
- H1, H10, H2, H3, H4, H5, H6, H7, H8, H9: value MOUNT_HOLE150MIL -> (none)
- J1: value 61400413321 -> (none)
- SW1, SW10, SW11, SW12, SW13, SW14, SW15, SW18, SW19, SW2, SW20, SW21, SW3, SW4, SW5, SW6, SW7, SW8, SW9: value B3W-9000-RG2C -> (none); device PP_Electromechanical:B3W-9000 -> PP_Electromechanical:MX1A
- SW16, SW17: value B3W-9000-RG2C -> (none); device PP_Electromechanical:B3W-9000 -> PP_Electromechanical:5501
- moved SW16 311.6 mm to (45.0, 30.0), turned to 90 degrees
- moved SW19 268.0 mm to (20.0, 90.0)
- moved SW21 151.8 mm to (140.0, 90.0)
- moved SW20 148.1 mm to (140.0, 125.0)
- moved SW18 123.7 mm to (20.0, 125.0)
- moved SW17 103.1 mm to (165.0, 30.0), turned to 90 degrees
- moved SW15 77.2 mm to (289.0, 13.0)
- moved U1 73.8 mm to (20.4, 59.1)
- moved SW14 55.9 mm to (289.0, 30.0)
- moved H9 47.2 mm to (260.0, 155.0)
- moved H10 40.0 mm to (140.0, 155.0)
- moved SW13 34.7 mm to (289.0, 47.0)
- moved DISP21 30.0 mm to (277.0, 122.0)
- moved SW9 28.6 mm to (289.0, 71.0)
- moved SW5 27.2 mm to (289.0, 88.0)
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Other:
- outline, holes or cut-outs redrawn
