File: Hardware/SSPS Front Panel/SSPS Front Panel.sch (EAGLE design)
At the start: 37 parts, among them U1 P8X32A-Q44

Commit message: figuring out LEDS
Parts:
- removed DISP17, DISP18, DISP19, DISP20, DISP21, DISP22, DISP23, DISP24, DISP25, DISP26, DISP27, DISP28, DISP29, DISP30, DISP31, DISP32: (no value), PP_LED:PSA08-11GWA
- removed DISP33, DISP34, DISP35: (no value), PP_LED:20SEG_LEDBARGRAPH
- added D1, D10, D11, D12, D13, D14, D15, D16, D2, D3, D4, D5, D6, D7, D8, D9: (no value), PP_LED:LED_SINGLE_WP1043
Changed lines of the file:
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@@
 <?xml version="1.0" encoding="utf-8"?>
 <!DOCTYPE eagle SYSTEM "eagle.dtd">
-<eagle version="6.5.0">
+<eagle version="6.6.0">
 <drawing>
 <settings>
@@
 <part name="DISP15" library="PP_LED" deviceset="PSA08-11GWA" device=""/>
 <part name="DISP16" library="PP_LED" deviceset="PSA08-11GWA" device=""/>
-<part name="DISP17" library="PP_LED" deviceset="PSA08-11GWA" device=""/>
-<part name="DISP18" library="PP_LED" deviceset="PSA08-11GWA" device=""/>
-<part name="DISP19" library="PP_LED" deviceset="PSA08-11GWA" device=""/>
-<part name="DISP20" library="PP_LED" deviceset="PSA08-11GWA" device=""/>
-<part name="DISP21" library="PP_LED" deviceset="PSA08-11GWA" device=""/>
-<part name="DISP22" library="PP_LED" deviceset="PSA08-11GWA" device=""/>
-<part name="DISP23" library="PP_LED" deviceset="PSA08-11GWA" device=""/>
-<part name="DISP24" library="PP_LED" deviceset="PSA08-11GWA" device=""/>
-<part name="DISP25" library="PP_LED" deviceset="PSA08-11GWA" device=""/>
-<part name="DISP26" library="PP_LED" deviceset="PSA08-11GWA" device=""/>
-<part name="DISP27" library="PP_LED" deviceset="PSA08-11GWA" device=""/>
-<part name="DISP28" library="PP_LED" deviceset="PSA08-11GWA" device=""/>
-<part name="DISP29" library="PP_LED" deviceset="PSA08-11GWA" device=""/>
-<part name="DISP30" library="PP_LED" deviceset="PSA08-11GWA" device=""/>
-<part name="DISP31" library="PP_LED" deviceset="PSA08-11GWA" device=""/>
-<part name="DISP32" library="PP_LED" deviceset="PSA08-11GWA" device=""/>
-<part name="DISP33" library="PP_LED" deviceset="20SEG_LEDBARGRAPH" device=""/>
-<part name="DISP34" library="PP_LED" deviceset="20SEG_LEDBARGRAPH" device=""/>
-<part name="DISP35" library="PP_LED" deviceset="20SEG_LEDBARGRAPH" device=""/>
 <part name="DISP36" library="PP_LED" deviceset="20SEG_LEDBARGRAPH" device=""/>
+<part name="D1" library="PP_LED" deviceset="LED_SINGLE" device="_WP1043"/>
+<part name="D2" library="PP_LED" deviceset="LED_SINGLE" device="_WP1043"/>
+<part name="D3" library="PP_LED" deviceset="LED_SINGLE" device="_WP1043"/>
+<part name="D4" library="PP_LED" deviceset="LED_SINGLE" device="_WP1043"/>
+<part name="D5" library="PP_LED" deviceset="LED_SINGLE" device="_WP1043"/>
+<part name="D6" library="PP_LED" deviceset="LED_SINGLE" device="_WP1043"/>
+<part name="D7" library="PP_LED" deviceset="LED_SINGLE" device="_WP1043"/>
+<part name="D8" library="PP_LED" deviceset="LED_SINGLE" device="_WP1043"/>
+<part name="D9" library="PP_LED" deviceset="LED_SINGLE" device="_WP1043"/>
+<part name="D10" library="PP_LED" deviceset="LED_SINGLE" device="_WP1043"/>
+<part name="D11" library="PP_LED" deviceset="LED_SINGLE" device="_WP1043"/>
+<part name="D12" library="PP_LED" deviceset="LED_SINGLE" device="_WP1043"/>
+<part name="D13" library="PP_LED" deviceset="LED_SINGLE" device="_WP1043"/>
+<part name="D14" library="PP_LED" deviceset="LED_SINGLE" device="_WP1043"/>
+<part name="D15" library="PP_LED" deviceset="LED_SINGLE" device="_WP1043"/>
+<part name="D16" library="PP_LED" deviceset="LED_SINGLE" device="_WP1043"/>
 </parts>
 <sheets>
@@
 <instance part="DISP15" gate="G$1" x="322.58" y="78.74"/>
 <instance part="DISP16" gate="G$1" x="322.58" y="43.18"/>
-<instance part="DISP17" gate="G$1" x="386.08" y="149.86"/>
-<instance part="DISP18" gate="G$1" x="386.08" y="114.3"/>
-<instance part="DISP19" gate="G$1" x="386.08" y="78.74"/>
-<instance part="DISP20" gate="G$1" x="386.08" y="43.18"/>
-<instance part="DISP21" gate="G$1" x="444.5" y="149.86"/>
-<instance part="DISP22" gate="G$1" x="444.5" y="114.3"/>
-<instance part="DISP23" gate="G$1" x="444.5" y="78.74"/>
-<instance part="DISP24" gate="G$1" x="444.5" y="43.18"/>
-<instance part="DISP25" gate="G$1" x="505.46" y="149.86"/>
-<instance part="DISP26" gate="G$1" x="505.46" y="114.3"/>
-<instance part="DISP27" gate="G$1" x="505.46" y="78.74"/>
-<instance part="DISP28" gate="G$1" x="505.46" y="43.18"/>
-<instance part="DISP29" gate="G$1" x="563.88" y="149.86"/>
-<instance part="DISP30" gate="G$1" x="563.88" y="114.3"/>
-<instance part="DISP31" gate="G$1" x="563.88" y="78.74"/>
-<instance part="DISP32" gate="G$1" x="563.88" y="43.18"/>
-<instance part="DISP33" gate="G$1" x="655.32" y="132.08"/>
-<instance part="DISP34" gate="G$1" x="675.64" y="132.08"/>
-<instance part="DISP35" gate="G$1" x="695.96" y="132.08"/>
 <instance part="DISP36" gate="G$1" x="716.28" y="132.08"/>
+<instance part="D1" gate="G$1" x="637.54" y="147.32"/>
+<instance part="D2" gate="G$1" x="637.54" y="134.62"/>
+<instance part="D3" gate="G$1" x="637.54" y="121.92"/>
+<instance part="D4" gate="G$1" x="637.54" y="109.22"/>
+<instance part="D5" gate="G$1" x="637.54" y="93.98"/>
+<instance part="D6" gate="G$1" x="637.54" y="81.28"/>
+<instance part="D7" gate="G$1" x="637.54" y="68.58"/>
+<instance part="D8" gate="G$1" x="637.54" y="55.88"/>
+<instance part="D9" gate="G$1" x="650.24" y="147.32"/>
+<instance part="D10" gate="G$1" x="650.24" y="134.62"/>
+<instance part="D11" gate="G$1" x="650.24" y="121.92"/>
+<instance part="D12" gate="G$1" x="650.24" y="109.22"/>
+<instance part="D13" gate="G$1" x="650.24" y="93.98"/>
+<instance part="D14" gate="G$1" x="650.24" y="81.28"/>
+<instance part="D15" gate="G$1" x="650.24" y="68.58"/>
+<instance part="D16" gate="G$1" x="650.24" y="55.88"/>
 </instances>
 <busses>

Commit message: Working on Front panel.
Parts:
- removed DISP36: (no value), PP_LED:20SEG_LEDBARGRAPH
- added D100, D101, D102, D103, D104, D105, D106, D107, D108, D17, D18, D19, D20, D21, D22, D23, D24, D25, D26, D27, D28, D29, D30, D31, D32, D33, D34, D35, D36, D37, D38, D39, D40, D41, D42, D43, D44, D45, D46, D47, D48, D49, D50, D51, D52, D53, D54, D55, D56, D57, D58, D59, D60, D61, D62, D63, D64, D65, D66, D67, D68, D69, D70, D71, D72, D73, D74, D75, D76, D77, D78, D79, D80, D81, D82, D83, D84, D85, D86, D87, D88, D89, D90, D91, D92, D93, D94, D95, D96, D97, D98, D99: (no value), PP_LED:LED_SINGLE_WP1043
- added DISP17, DISP18, DISP19, DISP20: PSA08-11GWA, PP_LED:PSA08-11GWA
- added SW1, SW10, SW11, SW12, SW13, SW14, SW15, SW16, SW2, SW3, SW4, SW5, SW6, SW7, SW8, SW9: B3W-9000-RG2C, PP_Electromechanical:B3W-9000
- DISP1, DISP10, DISP11, DISP12, DISP13, DISP14, DISP15, DISP16, DISP2, DISP3, DISP4, DISP5, DISP6, DISP7, DISP8, DISP9: value (none) -> PSA08-11GWA
Other:
- moved on the sheet: D10, D11, D12, D13, D14, D15, D16, D5, D6, D7, D8, D9

Commit message: Layout for front panel update.
Parts:
- added EN1, EN2: PEL12T-4226F-S1024, PP_Electromechanical:PEL12T
- added H1, H10, H2, H3, H4, H5, H6, H7, H8, H9: MOUNT_HOLE150MIL, PP_Connectors:MOUNT_HOLE150MIL
- added LCD1: (no value), PP_Displays:HD44780_LCD1602_COUNTERSINK
- added SW17, SW18, SW19, SW20, SW21, SW22, SW23, SW24: B3W-9000-RG2C, PP_Electromechanical:B3W-9000
- added SW25, SW26: 5501M112, PP_Electromechanical:5501

Commit message: Front panel test layout almost complete.
Parts:
- removed LCD1: (no value), PP_Displays:HD44780_LCD1602_COUNTERSINK
- removed SW24: B3W-9000-RG2C, PP_Electromechanical:B3W-9000
- added DISP21: CU16025-UWJ6, PP_Displays:CU16025-UWJ6
- added J1: 61400413321, PP_Connectors:USB_4PIN_61400413321
- added U2: STP16CP05XTTR, PP_DigitalIC:STP16CP05XTTR

Commit message: Working on front panel.
Parts:
- removed SW22, SW23: B3W-9000-RG2C, PP_Electromechanical:B3W-9000
- removed SW25, SW26: 5501M112, PP_Electromechanical:5501
- DISP1, DISP10, DISP11, DISP12, DISP13, DISP14, DISP15, DISP16, DISP17, DISP18, DISP19, DISP2, DISP20, DISP3, DISP4, DISP5, DISP6, DISP7, DISP8, DISP9: device PP_LED:PSA08-11GWA -> PP_LED:PSA08-11SRWA
- J1: value 61400413321 -> (none)
- SW1, SW10, SW11, SW12, SW13, SW14, SW15, SW18, SW19, SW2, SW20, SW21, SW3, SW4, SW5, SW6, SW7, SW8, SW9: value B3W-9000-RG2C -> (none); device PP_Electromechanical:B3W-9000 -> PP_Electromechanical:SPST_MX1A
- SW16, SW17: value B3W-9000-RG2C -> (none); device PP_Electromechanical:B3W-9000 -> PP_Electromechanical:5501
